Commit message: Raise neck mount by 15mm to match real robot hardware change
The neck mechanism was physically lifted 15mm on the real robot to
increase the head's range of motion. Updated head_fixed_joint origin
in the URDF to reflect this, keeping all neck/head kinematics unchanged.

File: garmi_description/urdf/garmi.urdf (robot description, URDF)
Before this commit: robot r100-0603, 64 links, 63 joints
Joints:
- joint head_fixed_joint: origin (none) -> xyz=0.0 0.0 0.015 rpy=0.0 0.0 0.0
