Commit message: Rename joints, TF frames and controllers to match the real robot
Align the model's names with the running Garmi so its /joint_states, TF and
controller topics line up with the real system:
- Arms: arm_0/arm_1 -> left_fr3_* / right_fr3_* (joints, links, hand and
  finger frames); URDF and MJCF now use identical names.
- Head: head_pan/tilt_joint -> o1_motor_1 / o1_motor_2 (the olive servo).
- Controllers: left_arm_joint_trajectory_controller,
  left_arm_joint_velocity_controller, lift_0_position_controller,
  platform_velocity_controller, head_controller.
Wheels and lift already matched. Mesh assets and the asset build script are
unaffected (mesh file names are unchanged).

File: garmi_description/urdf/garmi.urdf (robot description, URDF)
Before this commit: robot r100-0603, 64 links, 63 joints
Links:
- removed link arm_0_fr3_link0
- removed link arm_0_fr3_link1
- removed link arm_0_fr3_link2
- removed link arm_0_fr3_link3
- removed link arm_0_fr3_link4
- removed link arm_0_fr3_link5
- removed link arm_0_fr3_link6
- removed link arm_0_fr3_link7
- removed link arm_0_fr3_link8
- removed link arm_0_gripper_fr3_hand
- removed link arm_0_gripper_fr3_hand_tcp
- removed link arm_0_gripper_fr3_leftfinger
- removed link arm_0_gripper_fr3_rightfinger
- removed link arm_1_fr3_link0
- removed link arm_1_fr3_link1
- removed link arm_1_fr3_link2
- removed link arm_1_fr3_link3
- removed link arm_1_fr3_link4
- removed link arm_1_fr3_link5
- removed link arm_1_fr3_link6
- removed link arm_1_fr3_link7
- removed link arm_1_fr3_link8
- removed link arm_1_gripper_fr3_hand
- removed link arm_1_gripper_fr3_hand_tcp
- removed link arm_1_gripper_fr3_leftfinger
- removed link arm_1_gripper_fr3_rightfinger
- added link left_fr3_hand, mass 0.6544; collision mesh filename=package://garmi_description/meshes/hand.stl; visual mesh filename=package://garmi_description/meshes/hand.dae
- added link left_fr3_hand_tcp
- added link left_fr3_leftfinger, mass 0.0291; collision box size=17.5e-3 15.2e-3 18.5e-3; collision box size=17.5e-3 7e-3 23.5e-3
- added link left_fr3_link0, mass 2.3966; collision mesh filename=package://garmi_description/meshes/link0.stl; visual mesh filename=package://garmi_description/meshes/link0.dae
- added link left_fr3_link1, mass 2.9274653454; collision mesh filename=package://garmi_description/meshes/link1.stl; visual mesh filename=package://garmi_description/meshes/link1.dae
- added link left_fr3_link2, mass 2.9355370338; collision mesh filename=package://garmi_description/meshes/link2.stl; visual mesh filename=package://garmi_description/meshes/link2.dae
- added link left_fr3_link3, mass 2.2449013699; collision mesh filename=package://garmi_description/meshes/link3.stl; visual mesh filename=package://garmi_description/meshes/link3.dae
- added link left_fr3_link4, mass 2.6155955791; collision mesh filename=package://garmi_description/meshes/link4.stl; visual mesh filename=package://garmi_description/meshes/link4.dae
- added link left_fr3_link5, mass 2.3271207594; collision mesh filename=package://garmi_description/meshes/link5.stl; visual mesh filename=package://garmi_description/meshes/link5.dae
- added link left_fr3_link6, mass 1.8170376524; collision mesh filename=package://garmi_description/meshes/link6.stl; visual mesh filename=package://garmi_description/meshes/link6.dae
- added link left_fr3_link7, mass 0.6271432862; collision mesh filename=package://garmi_description/meshes/link7.stl; visual mesh filename=package://garmi_description/meshes/link7.dae
- added link left_fr3_link8
- added link left_fr3_rightfinger, mass 0.0291; collision box size=17.5e-3 15.2e-3 18.5e-3; collision box size=17.5e-3 7e-3 23.5e-3
- added link right_fr3_hand, mass 0.6544; collision mesh filename=package://garmi_description/meshes/hand.stl; visual mesh filename=package://garmi_description/meshes/hand.dae
- added link right_fr3_hand_tcp
- added link right_fr3_leftfinger, mass 0.0291; collision box size=17.5e-3 15.2e-3 18.5e-3; collision box size=17.5e-3 7e-3 23.5e-3
- added link right_fr3_link0, mass 2.3966; collision mesh filename=package://garmi_description/meshes/link0.stl; visual mesh filename=package://garmi_description/meshes/link0.dae
- added link right_fr3_link1, mass 2.9274653454; collision mesh filename=package://garmi_description/meshes/link1.stl; visual mesh filename=package://garmi_description/meshes/link1.dae
- added link right_fr3_link2, mass 2.9355370338; collision mesh filename=package://garmi_description/meshes/link2.stl; visual mesh filename=package://garmi_description/meshes/link2.dae
- added link right_fr3_link3, mass 2.2449013699; collision mesh filename=package://garmi_description/meshes/link3.stl; visual mesh filename=package://garmi_description/meshes/link3.dae
- added link right_fr3_link4, mass 2.6155955791; collision mesh filename=package://garmi_description/meshes/link4.stl; visual mesh filename=package://garmi_description/meshes/link4.dae
- added link right_fr3_link5, mass 2.3271207594; collision mesh filename=package://garmi_description/meshes/link5.stl; visual mesh filename=package://garmi_description/meshes/link5.dae
- added link right_fr3_link6, mass 1.8170376524; collision mesh filename=package://garmi_description/meshes/link6.stl; visual mesh filename=package://garmi_description/meshes/link6.dae
- added link right_fr3_link7, mass 0.6271432862; collision mesh filename=package://garmi_description/meshes/link7.stl; visual mesh filename=package://garmi_description/meshes/link7.dae
- added link right_fr3_link8
- added link right_fr3_rightfinger, mass 0.0291; collision box size=17.5e-3 15.2e-3 18.5e-3; collision box size=17.5e-3 7e-3 23.5e-3
Joints:
- removed joint arm_0_fr3_joint0
- removed joint arm_0_fr3_joint1
- removed joint arm_0_fr3_joint2
- removed joint arm_0_fr3_joint3
- removed joint arm_0_fr3_joint4
- removed joint arm_0_fr3_joint5
- removed joint arm_0_fr3_joint6
- removed joint arm_0_fr3_joint7
- removed joint arm_0_fr3_joint8
- removed joint arm_0_gripper_fr3_finger_joint1
- removed joint arm_0_gripper_fr3_finger_joint2
- removed joint arm_0_gripper_fr3_hand_joint
- removed joint arm_0_gripper_fr3_hand_tcp_joint
- removed joint arm_1_fr3_joint0
- removed joint arm_1_fr3_joint1
- removed joint arm_1_fr3_joint2
- removed joint arm_1_fr3_joint3
- removed joint arm_1_fr3_joint4
- removed joint arm_1_fr3_joint5
- removed joint arm_1_fr3_joint6
- removed joint arm_1_fr3_joint7
- removed joint arm_1_fr3_joint8
- removed joint arm_1_gripper_fr3_finger_joint1
- removed joint arm_1_gripper_fr3_finger_joint2
- removed joint arm_1_gripper_fr3_hand_joint
- removed joint arm_1_gripper_fr3_hand_tcp_joint
- removed joint head_pan_joint
- removed joint head_tilt_joint
- added joint left_fr3_finger_joint1: type prismatic, parent left_fr3_hand, child left_fr3_leftfinger, origin xyz=0 0 0.0584 rpy=0 0 0, axis 0 1 0, limit lower=0.0 upper=0.04 effort=100 velocity=0.2
- added joint left_fr3_finger_joint2: type prismatic, parent left_fr3_hand, child left_fr3_rightfinger, origin xyz=0 0 0.0584 rpy=0 0 3.141592653589793, axis 0 1 0, limit lower=0.0 upper=0.04 effort=100 velocity=0.2, mimic joint=left_fr3_finger_joint1
- added joint left_fr3_hand_joint: type fixed, parent left_fr3_link8, child left_fr3_hand, origin xyz=0 0 0 rpy=0 0 -0.7853981633974483
- added joint left_fr3_hand_tcp_joint: type fixed, parent left_fr3_hand, child left_fr3_hand_tcp, origin xyz=0 0 0.1034 rpy=0 0 0
- added joint left_fr3_joint0: type fixed, parent arm_mount_left_link, child left_fr3_link0, origin xyz=0.0 0.0 0.0 rpy=0.0 0.0 0.0
- added joint left_fr3_joint1: type revolute, parent left_fr3_link0, child left_fr3_link1, origin xyz=0 0 0.333 rpy=0 0 0, axis 0 0 1, limit lower=-2.9007 upper=2.9007 effort=87.0 velocity=2.62
- added joint left_fr3_joint2: type revolute, parent left_fr3_link1, child left_fr3_link2, origin xyz=0 0 0 rpy=-1.570796326794897 0 0, axis 0 0 1, limit lower=-1.8361 upper=1.8361 effort=87.0 velocity=2.62
- added joint left_fr3_joint3: type revolute, parent left_fr3_link2, child left_fr3_link3, origin xyz=0 -0.316 0 rpy=1.570796326794897 0 0, axis 0 0 1, limit lower=-2.9007 upper=2.9007 effort=87.0 velocity=2.62
- added joint left_fr3_joint4: type revolute, parent left_fr3_link3, child left_fr3_link4, origin xyz=0.0825 0 0 rpy=1.570796326794897 0 0, axis 0 0 1, limit lower=-3.077 upper=-0.1169 effort=87.0 velocity=2.62
- added joint left_fr3_joint5: type revolute, parent left_fr3_link4, child left_fr3_link5, origin xyz=-0.0825 0.384 0 rpy=-1.570796326794897 0 0, axis 0 0 1, limit lower=-2.8763 upper=2.8763 effort=12.0 velocity=5.26
- added joint left_fr3_joint6: type revolute, parent left_fr3_link5, child left_fr3_link6, origin xyz=0 0 0 rpy=1.570796326794897 0 0, axis 0 0 1, limit lower=0.4398 upper=4.6216 effort=12.0 velocity=4.18
- added joint left_fr3_joint7: type revolute, parent left_fr3_link6, child left_fr3_link7, origin xyz=0.088 0 0 rpy=1.570796326794897 0 0, axis 0 0 1, limit lower=-3.0508 upper=3.0508 effort=12.0 velocity=5.26
- added joint left_fr3_joint8: type fixed, parent left_fr3_link7, child left_fr3_link8, origin xyz=0 0 0.107 rpy=0 0 0
- added joint o1_motor_1: type revolute, parent neck_1, child neck_2, origin xyz=0.0279 0.0 0.0119 rpy=0.0 0.0 0.0, axis 0 0 1, limit lower=-1.5707 upper=1.5707 effort=30 velocity=1.5707
- added joint o1_motor_2: type revolute, parent neck_2, child head, origin xyz=0.0 -0.034 0.1521 rpy=0.0 0.0 0.0, axis 0 -1 0, limit lower=-0.7853 upper=0.7853 effort=30 velocity=1.5707
- added joint right_fr3_finger_joint1: type prismatic, parent right_fr3_hand, child right_fr3_leftfinger, origin xyz=0 0 0.0584 rpy=0 0 0, axis 0 1 0, limit lower=0.0 upper=0.04 effort=100 velocity=0.2
- added joint right_fr3_finger_joint2: type prismatic, parent right_fr3_hand, child right_fr3_rightfinger, origin xyz=0 0 0.0584 rpy=0 0 3.141592653589793, axis 0 1 0, limit lower=0.0 upper=0.04 effort=100 velocity=0.2, mimic joint=right_fr3_finger_joint1
- added joint right_fr3_hand_joint: type fixed, parent right_fr3_link8, child right_fr3_hand, origin xyz=0 0 0 rpy=0 0 -0.7853981633974483
- added joint right_fr3_hand_tcp_joint: type fixed, parent right_fr3_hand, child right_fr3_hand_tcp, origin xyz=0 0 0.1034 rpy=0 0 0
- added joint right_fr3_joint0: type fixed, parent arm_mount_right_link, child right_fr3_link0, origin xyz=0.0 0.0 0.0 rpy=0.0 0.0 0.0
- added joint right_fr3_joint1: type revolute, parent right_fr3_link0, child right_fr3_link1, origin xyz=0 0 0.333 rpy=0 0 0, axis 0 0 1, limit lower=-2.9007 upper=2.9007 effort=87.0 velocity=2.62
- added joint right_fr3_joint2: type revolute, parent right_fr3_link1, child right_fr3_link2, origin xyz=0 0 0 rpy=-1.570796326794897 0 0, axis 0 0 1, limit lower=-1.8361 upper=1.8361 effort=87.0 velocity=2.62
- added joint right_fr3_joint3: type revolute, parent right_fr3_link2, child right_fr3_link3, origin xyz=0 -0.316 0 rpy=1.570796326794897 0 0, axis 0 0 1, limit lower=-2.9007 upper=2.9007 effort=87.0 velocity=2.62
- added joint right_fr3_joint4: type revolute, parent right_fr3_link3, child right_fr3_link4, origin xyz=0.0825 0 0 rpy=1.570796326794897 0 0, axis 0 0 1, limit lower=-3.077 upper=-0.1169 effort=87.0 velocity=2.62
- added joint right_fr3_joint5: type revolute, parent right_fr3_link4, child right_fr3_link5, origin xyz=-0.0825 0.384 0 rpy=-1.570796326794897 0 0, axis 0 0 1, limit lower=-2.8763 upper=2.8763 effort=12.0 velocity=5.26
- added joint right_fr3_joint6: type revolute, parent right_fr3_link5, child right_fr3_link6, origin xyz=0 0 0 rpy=1.570796326794897 0 0, axis 0 0 1, limit lower=0.4398 upper=4.6216 effort=12.0 velocity=4.18
- added joint right_fr3_joint7: type revolute, parent right_fr3_link6, child right_fr3_link7, origin xyz=0.088 0 0 rpy=1.570796326794897 0 0, axis 0 0 1, limit lower=-3.0508 upper=3.0508 effort=12.0 velocity=5.26
- added joint right_fr3_joint8: type fixed, parent right_fr3_link7, child right_fr3_link8, origin xyz=0 0 0.107 rpy=0 0 0

Commit message: Collide the torso, cover, neck and head as convex proxies
* Problem: the torso, base cover, mounting plate, neck and head collided as their visual
  meshes, up to 100k triangles each, so every collision check against them was slow.
* Impact: each now collides as a convex proxy of ~1200 triangles that encloses the part and
  reaches at most 4.4 mm beyond its hull; the MuJoCo arms collide against the same proxies
  instead of three coarse boxes.
* Why this way: the proxies are garmi-core's true-size ones, byte for byte, under the same
  meshes/collision/ names, so the internal model can consume them; its inflated planning
  variants stay internal.
* Verification: every visual vertex lies inside its proxy (worst -0.14 mm); scene.xml loads with
  no non-floor contact in the home pose and none between body proxies over 400 head/lift poses.

File: garmi_description/urdf/garmi.urdf (robot description, URDF)
Before this commit: robot r100-0603, 64 links, 63 joints
Links:
- link body_link: geometry collision mesh filename=package://garmi_description/meshes/collision/body.stl; visual mesh filename=package://garmi_description/meshes/body.obj
- link cover_link: geometry collision mesh filename=package://garmi_description/meshes/collision/cover.stl; visual mesh filename=package://garmi_description/meshes/cover.obj
- link head: geometry collision mesh filename=package://garmi_description/meshes/collision/head.stl; visual mesh filename=package://garmi_description/meshes/head.obj
- link mounting_plate_link: geometry collision mesh filename=package://garmi_description/meshes/collision/mounting_plate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; visual mesh filename=package://garmi_description/meshes/mounting_plate.obj
- link neck_1: geometry collision mesh filename=package://garmi_description/meshes/collision/neck_1.stl; visual mesh filename=package://garmi_description/meshes/neck_1.obj
- link neck_2: geometry collision mesh filename=package://garmi_description/meshes/collision/neck_2.stl; visual mesh filename=package://garmi_description/meshes/neck_2.obj

Commit message: Add Garmi's long fingertips and move the TCP between them
* Problem: the model carried Franka's stock 17.8 mm fingertips, while the robot grips with 70 mm
  tips, so the hands were too short and the tool centre sat 26 mm behind the real pads.
* Impact: each finger gains a `<side>_fr3_<finger>_tip` link (box collision, wedge visual, 6.3 g)
  and `<side>_fr3_hand_tcp` moves from 103.4 to 129.5 mm; MuJoCo gets the same tips, replacing
  menagerie's stock pads that lie inside them, and a TCP site.
* Verification: link names, frames, geometry and inertials match garmi-core's expanded
  description exactly; in MuJoCo the TCP site sits on the two pads' midpoint and a gripper
  closes cleanly onto its own tips.

File: garmi_description/urdf/garmi.urdf (robot description, URDF)
Before this commit: robot r100-0603, 64 links, 63 joints
Links:
- added link left_fr3_leftfinger_tip, mass 0.00628; collision box size=0.0178 0.0109 0.07; visual mesh filename=package://garmi_description/meshes/fingertip.stl
- added link left_fr3_rightfinger_tip, mass 0.00628; collision box size=0.0178 0.0109 0.07; visual mesh filename=package://garmi_description/meshes/fingertip.stl
- added link right_fr3_leftfinger_tip, mass 0.00628; collision box size=0.0178 0.0109 0.07; visual mesh filename=package://garmi_description/meshes/fingertip.stl
- added link right_fr3_rightfinger_tip, mass 0.00628; collision box size=0.0178 0.0109 0.07; visual mesh filename=package://garmi_description/meshes/fingertip.stl
Joints:
- added joint left_fr3_leftfinger_tip_joint: type fixed, parent left_fr3_leftfinger, child left_fr3_leftfinger_tip, origin xyz=0 0 0.0711 rpy=0 0 0
- added joint left_fr3_rightfinger_tip_joint: type fixed, parent left_fr3_rightfinger, child left_fr3_rightfinger_tip, origin xyz=0 0 0.0711 rpy=0 0 0
- added joint right_fr3_leftfinger_tip_joint: type fixed, parent right_fr3_leftfinger, child right_fr3_leftfinger_tip, origin xyz=0 0 0.0711 rpy=0 0 0
- added joint right_fr3_rightfinger_tip_joint: type fixed, parent right_fr3_rightfinger, child right_fr3_rightfinger_tip, origin xyz=0 0 0.0711 rpy=0 0 0
- joint left_fr3_hand_tcp_joint: origin xyz=0 0 0.1034 rpy=0 0 0 -> xyz=0 0 0.1295 rpy=0 0 0
- joint right_fr3_hand_tcp_joint: origin xyz=0 0 0.1034 rpy=0 0 0 -> xyz=0 0 0.1295 rpy=0 0 0

Commit message: Add the Olive stereo camera on top of the head
* Problem: the head's stereo camera, its housing and stand were missing, so the model had no
  frames for the head's images and nothing for the arms to avoid on top of the head.
* Impact: `head_camera_mount`, `olive_camera_link`, `olive_camera_housing` and one optical frame
  per lens (63.0 mm baseline) ride the head; MuJoCo renders through one camera per lens.
* Why this way: the camera's pose on the adjustable stand stays garmi-core's best guess from
  photos (pitched down 10 degrees) rather than a measured one, flagged as such in the URDF.
* Verification: names, frames and geometry match garmi-core's expansion; the MuJoCo cameras sit
  on the URDF optical frames to 0.001 mm, and 400 head/lift poses give no body-on-body contact.

File: garmi_description/urdf/garmi.urdf (robot description, URDF)
Before this commit: robot r100-0603, 68 links, 67 joints
Links:
- added link head_camera_mount; collision cylinder length=0.03 radius=0.011; visual cylinder length=0.008 radius=0.004
- added link olive_camera_housing; visual mesh filename=package://garmi_description/meshes/olive_camera_housing.stl
- added link olive_camera_left_optical_frame
- added link olive_camera_link; collision mesh filename=package://garmi_description/meshes/collision/olive_camera.s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; visual mesh filename=package://garmi_description/meshes/olive_camera.stl
- added link olive_camera_right_optical_frame
Joints:
- added joint head_camera_mount_joint: type fixed, parent head, child head_camera_mount, origin xyz=0.0614 0.034 0.09 rpy=0 0 0
- added joint olive_camera_housing_joint: type fixed, parent olive_camera_link, child olive_camera_housing, origin xyz=0 0 0 rpy=0 0 0
- added joint olive_camera_joint: type fixed, parent head_camera_mount, child olive_camera_link, origin xyz=0.005 0 0.051 rpy=0 0.174533 0
- added joint olive_camera_left_optical_joint: type fixed, parent olive_camera_link, child olive_camera_left_optical_frame, origin xyz=0 0.0315 0 rpy=-1.5707963267948966 0 -1.5707963267948966
- added joint olive_camera_right_optical_joint: type fixed, parent olive_camera_link, child olive_camera_right_optical_frame, origin xyz=0 -0.0315 0 rpy=-1.5707963267948966 0 -1.5707963267948966
