Commit message: Add the wrist cameras on their brackets
* Problem: each hand carries a RealSense D435i on a 3D-printed bracket, but the model had
  neither, so the camera driver's frames had no transforms and the arms nothing to avoid.
* Impact: `<side>_fr3_wrist_camera_mount` (71.7 g) and the whole `camera_d435i_<side>_*` frame
  tree, optical frames included, ride each flange; MuJoCo renders through each colour sensor.
  The camera looks like the real one: grey housing, black glass front, charcoal lenses.
* Why this way: the camera's inertia is its collision box's, not the vendor model's placeholder,
  which is 70 times too large and would dwarf the hand's; mass and every frame stay the vendor's.
  The look is Intel's mesh with its triangles sorted into three materials and thinned out (15.8
  MB to 466 KB, `d435_garmi.dae`), plus the three parts as STLs, since MuJoCo reads no colours
  from a mesh; NOTICE and THIRD_PARTY_LICENSES now say the mesh is modified.
* Verification: all 103 links and 102 joints match garmi-core's expanded description in name,
  frame, geometry and inertia, with no exception; the MuJoCo model compiles and its frames
  match the URDF's to 0.001 mm.

File: garmi_description/urdf/garmi.urdf (robot description, URDF)
Before this commit: robot r100-0603, 73 links, 72 joints
Links:
- added link camera_d435i_left_accel_frame
- added link camera_d435i_left_accel_optical_frame
- added link camera_d435i_left_bottom_screw_frame
- added link camera_d435i_left_color_frame
- added link camera_d435i_left_color_optical_frame
- added link camera_d435i_left_depth_frame
- added link camera_d435i_left_depth_optical_frame
- added link camera_d435i_left_gyro_frame
- added link camera_d435i_left_gyro_optical_frame
- added link camera_d435i_left_infra1_frame
- added link camera_d435i_left_infra1_optical_frame
- added link camera_d435i_left_infra2_frame
- added link camera_d435i_left_infra2_optical_frame
- added link camera_d435i_left_link, mass 0.072; collision box size=0.02505 0.09 0.025; visual mesh filename=package://garmi_description/meshes/d435_garmi.dae
- added link camera_d435i_right_accel_frame
- added link camera_d435i_right_accel_optical_frame
- added link camera_d435i_right_bottom_screw_frame
- added link camera_d435i_right_color_frame
- added link camera_d435i_right_color_optical_frame
- added link camera_d435i_right_depth_frame
- added link camera_d435i_right_depth_optical_frame
- added link camera_d435i_right_gyro_frame
- added link camera_d435i_right_gyro_optical_frame
- added link camera_d435i_right_infra1_frame
- added link camera_d435i_right_infra1_optical_frame
- added link camera_d435i_right_infra2_frame
- added link camera_d435i_right_infra2_optical_frame
- added link camera_d435i_right_link, mass 0.072; collision box size=0.02505 0.09 0.025; visual mesh filename=package://garmi_description/meshes/d435_garmi.dae
- added link left_fr3_wrist_camera_mount, mass 0.0717; collision mesh filename=package://garmi_description/meshes/collision/wrist_camera_m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; visual mesh filename=package://garmi_description/meshes/wrist_camera_mount.stl
- added link right_fr3_wrist_camera_mount, mass 0.0717; collision mesh filename=package://garmi_description/meshes/collision/wrist_camera_m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; visual mesh filename=package://garmi_description/meshes/wrist_camera_mount.stl
Joints:
- added joint camera_d435i_left_accel_joint: type fixed, parent camera_d435i_left_link, child camera_d435i_left_accel_frame, origin xyz=-0.01174 -0.00552 0.0051 rpy=0 0 0
- added joint camera_d435i_left_accel_optical_joint: type fixed, parent camera_d435i_left_accel_frame, child camera_d435i_left_accel_optical_frame, origin xyz=0 0 0 rpy=-1.5707963267948966 0 -1.5707963267948966
- added joint camera_d435i_left_color_joint: type fixed, parent camera_d435i_left_link, child camera_d435i_left_color_frame, origin xyz=0 0.015 0 rpy=0 0 0
- added joint camera_d435i_left_color_optical_joint: type fixed, parent camera_d435i_left_color_frame, child camera_d435i_left_color_optical_frame, origin xyz=0 0 0 rpy=-1.5707963267948966 0 -1.5707963267948966
- added joint camera_d435i_left_depth_joint: type fixed, parent camera_d435i_left_link, child camera_d435i_left_depth_frame, origin xyz=0 0 0 rpy=0 0 0
- added joint camera_d435i_left_depth_optical_joint: type fixed, parent camera_d435i_left_depth_frame, child camera_d435i_left_depth_optical_frame, origin xyz=0 0 0 rpy=-1.5707963267948966 0 -1.5707963267948966
- added joint camera_d435i_left_gyro_joint: type fixed, parent camera_d435i_left_link, child camera_d435i_left_gyro_frame, origin xyz=-0.01174 -0.00552 0.0051 rpy=0 0 0
- added joint camera_d435i_left_gyro_optical_joint: type fixed, parent camera_d435i_left_gyro_frame, child camera_d435i_left_gyro_optical_frame, origin xyz=0 0 0 rpy=-1.5707963267948966 0 -1.5707963267948966
- added joint camera_d435i_left_infra1_joint: type fixed, parent camera_d435i_left_link, child camera_d435i_left_infra1_frame, origin xyz=0 0.0 0 rpy=0 0 0
- added joint camera_d435i_left_infra1_optical_joint: type fixed, parent camera_d435i_left_infra1_frame, child camera_d435i_left_infra1_optical_frame, origin xyz=0 0 0 rpy=-1.5707963267948966 0 -1.5707963267948966
- added joint camera_d435i_left_infra2_joint: type fixed, parent camera_d435i_left_link, child camera_d435i_left_infra2_frame, origin xyz=0 -0.05 0 rpy=0 0 0
- added joint camera_d435i_left_infra2_optical_joint: type fixed, parent camera_d435i_left_infra2_frame, child camera_d435i_left_infra2_optical_frame, origin xyz=0 0 0 rpy=-1.5707963267948966 0 -1.5707963267948966
- added joint camera_d435i_left_joint: type fixed, parent left_fr3_wrist_camera_mount, child camera_d435i_left_bottom_screw_frame, origin xyz=0.11001 0.0 0.02231 rpy=0 -0.7853981633974483 3.141592653589793
- added joint camera_d435i_left_link_joint: type fixed, parent camera_d435i_left_bottom_screw_frame, child camera_d435i_left_link, origin xyz=0.010600000000000002 0.0175 0.0125 rpy=0 0 0
- added joint camera_d435i_right_accel_joint: type fixed, parent camera_d435i_right_link, child camera_d435i_right_accel_frame, origin xyz=-0.01174 -0.00552 0.0051 rpy=0 0 0
- added joint camera_d435i_right_accel_optical_joint: type fixed, parent camera_d435i_right_accel_frame, child camera_d435i_right_accel_optical_frame, origin xyz=0 0 0 rpy=-1.5707963267948966 0 -1.5707963267948966
- added joint camera_d435i_right_color_joint: type fixed, parent camera_d435i_right_link, child camera_d435i_right_color_frame, origin xyz=0 0.015 0 rpy=0 0 0
- added joint camera_d435i_right_color_optical_joint: type fixed, parent camera_d435i_right_color_frame, child camera_d435i_right_color_optical_frame, origin xyz=0 0 0 rpy=-1.5707963267948966 0 -1.5707963267948966
- added joint camera_d435i_right_depth_joint: type fixed, parent camera_d435i_right_link, child camera_d435i_right_depth_frame, origin xyz=0 0 0 rpy=0 0 0
- added joint camera_d435i_right_depth_optical_joint: type fixed, parent camera_d435i_right_depth_frame, child camera_d435i_right_depth_optical_frame, origin xyz=0 0 0 rpy=-1.5707963267948966 0 -1.5707963267948966
- added joint camera_d435i_right_gyro_joint: type fixed, parent camera_d435i_right_link, child camera_d435i_right_gyro_frame, origin xyz=-0.01174 -0.00552 0.0051 rpy=0 0 0
- added joint camera_d435i_right_gyro_optical_joint: type fixed, parent camera_d435i_right_gyro_frame, child camera_d435i_right_gyro_optical_frame, origin xyz=0 0 0 rpy=-1.5707963267948966 0 -1.5707963267948966
- added joint camera_d435i_right_infra1_joint: type fixed, parent camera_d435i_right_link, child camera_d435i_right_infra1_frame, origin xyz=0 0.0 0 rpy=0 0 0
- added joint camera_d435i_right_infra1_optical_joint: type fixed, parent camera_d435i_right_infra1_frame, child camera_d435i_right_infra1_optical_frame, origin xyz=0 0 0 rpy=-1.5707963267948966 0 -1.5707963267948966
- added joint camera_d435i_right_infra2_joint: type fixed, parent camera_d435i_right_link, child camera_d435i_right_infra2_frame, origin xyz=0 -0.05 0 rpy=0 0 0
- added joint camera_d435i_right_infra2_optical_joint: type fixed, parent camera_d435i_right_infra2_frame, child camera_d435i_right_infra2_optical_frame, origin xyz=0 0 0 rpy=-1.5707963267948966 0 -1.5707963267948966
- added joint camera_d435i_right_joint: type fixed, parent right_fr3_wrist_camera_mount, child camera_d435i_right_bottom_screw_frame, origin xyz=0.11001 0.0 0.02231 rpy=0 -0.7853981633974483 3.141592653589793
- added joint camera_d435i_right_link_joint: type fixed, parent camera_d435i_right_bottom_screw_frame, child camera_d435i_right_link, origin xyz=0.010600000000000002 0.0175 0.0125 rpy=0 0 0
- added joint left_fr3_wrist_camera_mount_joint: type fixed, parent left_fr3_link8, child left_fr3_wrist_camera_mount, origin xyz=0 0 0 rpy=0 0 -0.7853981633974483
- added joint right_fr3_wrist_camera_mount_joint: type fixed, parent right_fr3_link8, child right_fr3_wrist_camera_mount, origin xyz=0 0 0 rpy=0 0 -0.7853981633974483

Commit message: Seat the head camera on its printed mount
* Problem: the head camera stood on a provisional stand in Olive's housing, a pose guessed from
  photos, while the robot now carries it in a printed housing and lens cover on a printed mount
  whose foot replaces the inlay on top of the head.
* Impact: the mount, housing and cover are the technician's CAD, the head's mesh loses its inlay,
  and `olive_camera_link` with both optical frames sits on the cover's two lens openings
  (63.0 mm apart, 11.66 degrees down); names are unchanged.
* Why this way: garmi-core's scripts/head_camera_mount_mesh.py writes the meshes and drops the
  inlay from the STEP, so both can be made again; the STEP itself is not shipped.
* Verification: garmi-core's description tests pass on this model; the MuJoCo cameras sit on the
  URDF optical frames to 0.0001 mm, and 400 head/lift poses give no body-on-body contact.

File: garmi_description/urdf/garmi.urdf (robot description, URDF)
Before this commit: robot r100-0603, 103 links, 102 joints
Links:
- link head_camera_mount: mass None -> 0.01525; geometry collision mesh filename=package://garmi_description/meshes/collision/head_camera_mo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; visual mesh filename=package://garmi_description/meshes/head_camera_mount.stl
- link olive_camera_housing: mass None -> 0.02245; geometry visual mesh filename=package://garmi_description/meshes/olive_camera_cover.stl; visual mesh filename=package://garmi_description/meshes/olive_camera_housing.stl
Joints:
- joint head_camera_mount_joint: origin xyz=0.0614 0.034 0.09 rpy=0 0 0 -> xyz=0.0459 0.034 0.09 rpy=0 0 0
- joint olive_camera_joint: origin xyz=0.005 0 0.051 rpy=0 0.174533 0 -> xyz=0.020651 -0.00002 0.027986 rpy=0 0.203511 -0.000096

Commit message: Draw the neck's pan-tilt unit from its CAD
* Problem: the neck was drawn from the design meshes, its 15 mm taller base modelled as a raise of the
  whole neck, which lifted the base's flange up to 7 mm into the torso's collar.
* Impact: `neck_1`, `neck_2` and a second head visual draw the technician's gimbal (motors as the CAD's
  plain cylinders); the raise moves to `o1_motor_1`, so `neck_1` sits 15 mm lower while `neck_2`, the
  head and its camera keep their poses.
* Why this way: garmi-core's scripts/head_gimbal_mesh.py writes meshes and proxies from the STEP, which
  is not shipped.
* Verification: `check_urdf` parses; in MuJoCo the head cameras sit on the URDF optical frames, and
  634 head/lift poses give no body-on-body contact.

File: garmi_description/urdf/garmi.urdf (robot description, URDF)
Before this commit: robot r100-0603, 103 links, 102 joints
Links:
- link head: geometry collision mesh filename=package://garmi_description/meshes/collision/head.stl; visual mesh filename=package://garmi_description/meshes/head.obj
Joints:
- joint head_fixed_joint: origin xyz=0.0 0.0 0.015 rpy=0.0 0.0 0.0 -> xyz=0.0 0.0 0.0 rpy=0.0 0.0 0.0
- joint o1_motor_1: origin xyz=0.0279 0.0 0.0119 rpy=0.0 0.0 0.0 -> xyz=0.0279 0.0 0.0269 rpy=0.0 0.0 0.0

Commit message: Turn the head's pan and tilt the way the real head does
* Problem: both Olive servo joints had the wrong sign, so the model's head turned and nodded
  opposite to the real one for the same joint state (confirmed on the robot).
* Impact: `o1_motor_1` (pan) turns about 0 0 -1 and `o1_motor_2` (tilt) about 0 1 0, in the URDF
  and the MuJoCo model; names, symmetric limits and every frame at zero pan and tilt are unchanged.
* Verification: check_urdf parses; the MuJoCo scene loads with the new axes.

File: garmi_description/urdf/garmi.urdf (robot description, URDF)
Before this commit: robot r100-0603, 103 links, 102 joints
Joints:
- joint o1_motor_1: axis 0 0 1 -> 0 0 -1
- joint o1_motor_2: axis 0 -1 0 -> 0 1 0

Commit message: Seat the wrist cameras on the bracket's offset hole pair
* Problem: both wrist cameras are screwed to the bracket's offset hole pair, which puts each colour lens in its
  gripper's plane of symmetry, but the model seated them on the centered pair, 32.5 mm to the side.
* Impact: every camera_d435i_<side>_* frame moves 32.5 mm along the camera's long axis; the bracket's collision
  proxy is collision/wrist_camera_mount_offset.stl, replacing _centered. Link and joint names are unchanged.
* Verification: the colour optical frame sits at (111.354, 0.000, 38.644) mm in <side>_fr3_hand, in the URDF and in
  MuJoCo alike (0.0000 mm apart); the MuJoCo model compiles with no body-on-body contact at home.

File: garmi_description/urdf/garmi.urdf (robot description, URDF)
Before this commit: robot r100-0603, 103 links, 102 joints
Joints:
- joint camera_d435i_left_joint: origin xyz=0.11001 0.0 0.02231 rpy=0 -0.7853981633974483 3.141592653589793 -> xyz=0.11001 0.0325 0.02231 rpy=0 -0.7853981633974483 3.141592653589793
- joint camera_d435i_right_joint: origin xyz=0.11001 0.0 0.02231 rpy=0 -0.7853981633974483 3.141592653589793 -> xyz=0.11001 0.0325 0.02231 rpy=0 -0.7853981633974483 3.141592653589793
